File: Hardware/LibreCAL/Power.kicad_sch (KiCad schematic)
At the start: 7 parts, among them U9 MIC5528-3.3YMT-TR

Commit message: Improvements on LibreCAL KiCad: fixed minor errors/labels(cosmetic), improved BOM(Added LCSC_Part), improved Impedance JLCPCB 4Layer JLC7628 1.6mm
Parts:
- C28, C29, C32: LCSC_Part (none) -> C307418
- C30, C31: LCSC_Part (none) -> C307331
- FB2: LCSC_Part (none) -> C404693
- U9: LCSC_Part (none) -> C622490
Other:
- title: (none) -> LibreCAL
Changed lines of the file:
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@@
 (kicad_sch (version 20211123) (generator eeschema)
   (paper "A4")
+  (title_block
+    (title "LibreCAL")
+    (date "2023-01-07")
+    (rev "A+")
+  )
   (junction (at 119.38 90.17) (diameter 0) (color 0 0 0 0)
   )
@@
     )
     (property "Datasheet" "~" (id 3) (at 167.64 96.52 0)
+      (effects (font (size 1.27 1.27)) hide)
+    )
+    (property "LCSC_Part" "C307331" (id 4) (at 167.64 96.52 0)
       (effects (font (size 1.27 1.27)) hide)
     )
@@
     )
     (property "Datasheet" "~" (id 3) (at 107.95 96.52 0)
+      (effects (font (size 1.27 1.27)) hide)
+    )
+    (property "LCSC_Part" "C307418" (id 4) (at 107.95 96.52 0)
       (effects (font (size 1.27 1.27)) hide)
     )
@@
     )
     (property "Datasheet" "https://eu.mouser.com/datasheet/2/268/MIC5528_High_Performance_500mA_LDO_in_Thin_and_Ext-1891284.pdf" (id 3) (at 149.86 95.25 0)
+      (effects (font (size 1.27 1.27)) hide)
+    )
+    (property "LCSC_Part" "C622490" (id 4) (at 152.4 92.71 0)
       (effects (font (size 1.27 1.27)) hide)
     )
@@
       (effects (font (size 1.27 1.27)) hide)
     )
+    (property "LCSC_Part" "C307418" (id 4) (at 119.38 96.52 0)
+      (effects (font (size 1.27 1.27)) hide)
+    )
     (pin "1")
     (pin "2")
@@
     )
     (property "Datasheet" "~" (id 3) (at 180.34 96.52 0)
+      (effects (font (size 1.27 1.27)) hide)
+    )
+    (property "LCSC_Part" "C307418" (id 4) (at 180.34 96.52 0)
       (effects (font (size 1.27 1.27)) hide)
     )
@@
     )
     (property "Datasheet" "~" (id 3) (at 130.81 96.52 0)
+      (effects (font (size 1.27 1.27)) hide)
+    )
+    (property "LCSC_Part" "C307331" (id 4) (at 130.81 96.52 0)
       (effects (font (size 1.27 1.27)) hide)
     )
@@
       (effects (font (size 1.27 1.27)) hide)
     )
+    (property "LCSC_Part" "C404693" (id 4) (at 102.87 90.17 0)
+      (effects (font (size 1.27 1.27)) hide)
+    )
